File: ESP32-BOBOARD-5V.sch (KiCad schematic (older format))
At the start: 27 parts, among them J1 Conn_01x15, J2 Conn_01x15, J3 Conn_02x16_Counter_Clockwise, J4 Conn_01x03_Male, J5 DX07S016JA1R1500, U1 TXS0108EPW, U3 TXS0108EPW, U4 TXS0108EPW

Commit message: Added the dip-switch for programming Added the ESP32 BOBOARD LOGO
Parts:
- added GR2: LOGO, RetroBitLab:ESP32_BOBOARD_5V_21.7mmx21.7mm, symbol RetroBitLab:LOGO
- added SW1: SPST_SWITCH_SMD_4P,4.1x5.4mm, RetroBitLab:SW_DIP_SPSTx02_DSHP02TS-S, symbol RetroBitLab:SPST_SWITCH_SMD_4P,4.1x5.4mm
- renumbered L1 to GR1
Connections:
- net labels added: TXS_EN
- wire segments 198 -> 204
- no-connect marks 8 -> 10
Other:
- note added: "Normal Mode\nOFF-OFF\nWhen PROGRAMMING ESP32\nON-ON"
- moved on the sheet: J3

Commit message: Updated to reflect new components from library and LCSC availability
Parts:
- removed C1, C2, C3, C4, C5, C6, C7, C8, C9: 100uF, Capacitor_SMD:C_1210_3225Metric_Pad1.33x2.70mm_HandSolder, symbol Device:C_Small
- removed C10: 100nF, Capacitor_SMD:C_1210_3225Metric_Pad1.33x2.70mm_HandSolder, symbol Device:C_Small
- removed R1, R2, R3, R4: 10K, Resistor_SMD:R_1210_3225Metric_Pad1.30x2.65mm_HandSolder, symbol Device:R_Small_US
- removed R5, R6: 5.1K, Resistor_SMD:R_1210_3225Metric_Pad1.30x2.65mm_HandSolder, symbol Device:R_Small_US
- removed R7, R8: 0R, Resistor_SMD:R_1210_3225Metric_Pad1.30x2.65mm_HandSolder, symbol Device:R_Small_US
- added C1, C2, C3, C4, C5, C6, C7, C8, C9: 100uF, Capacitor_SMD:C_1210_3225Metric_Pad1.33x2.70mm_HandSolder, symbol CCAP1210:100uF
- added C10: 100nF, Capacitor_SMD:C_1210_3225Metric_Pad1.33x2.70mm_HandSolder, symbol CCAP1210:100nF
- added R1, R2, R3, R4: 10K, Resistor_SMD:R_1210_3225Metric_Pad1.30x2.65mm_HandSolder, symbol CRES1210:10K
- added R5, R6: 5K1, Resistor_SMD:R_1210_3225Metric_Pad1.30x2.65mm_HandSolder, symbol CRES1210:5K1
- added R7, R8: CREZ12101%, Resistor_SMD:R_1210_3225Metric_Pad1.30x2.65mm_HandSolder, symbol CRES1210:CREZ12101%
Connections:
- wire segments 204 -> 210

Commit message: From 1210 to 0805 as the first are pretty hard to find nowadays.
Parts:
- removed C1, C2, C3, C4, C5, C6, C7, C8, C9: 100uF, Capacitor_SMD:C_1210_3225Metric_Pad1.33x2.70mm_HandSolder, symbol CCAP1210:100uF
- removed C10: 100nF, Capacitor_SMD:C_1210_3225Metric_Pad1.33x2.70mm_HandSolder, symbol CCAP1210:100nF
- removed J3: Conn_02x16_Counter_Clockwise, Connector_PinHeader_2.54mm:PinHeader_2x16_P2.54mm_Vertical_SMD, symbol Connector_Generic:Conn_02x16_Counter_Clockwise
- removed R1, R2, R3, R4: 10K, Resistor_SMD:R_1210_3225Metric_Pad1.30x2.65mm_HandSolder, symbol CRES1210:10K
- removed R5, R6: 5K1, Resistor_SMD:R_1210_3225Metric_Pad1.30x2.65mm_HandSolder, symbol CRES1210:5K1
- removed R7, R8: CREZ12101%, Resistor_SMD:R_1210_3225Metric_Pad1.30x2.65mm_HandSolder, symbol CRES1210:CREZ12101%
- added C1, C2, C3, C4, C5, C6, C7, C8, C9: 100uF, Capacitor_SMD:C_0805_2012Metric_Pad1.18x1.45mm_HandSolder, symbol CCAP0805:100uF
- added C10: 100nF, Capacitor_SMD:C_0805_2012Metric_Pad1.18x1.45mm_HandSolder, symbol CCAP0805:100nF
- added J3: CONN_02x16_PIN_SMD_Counter_Clockwise, Connector_PinHeader_2.54mm:PinHeader_2x16_P2.54mm_Vertical_SMD, symbol RetroBitLab:CONN_02x16_PIN_SMD_Counter_Clockwise
- added R1, R2, R3, R4: 10K, Resistor_SMD:R_0805_2012Metric_Pad1.20x1.40mm_HandSolder, symbol CRES0805:10K
- added R5, R6: 5K1, Resistor_SMD:R_0805_2012Metric_Pad1.20x1.40mm_HandSolder, symbol CRES0805:5K1
- added R7, R8: CREZ08051%, Resistor_SMD:R_0805_2012Metric_Pad1.20x1.40mm_HandSolder, symbol CRES0805:CREZ08051%
