File: ESP32-BOBOARD-5V.sch (KiCad schematic (older format))
At the start: 29 parts, among them J1 Conn_01x15, J2 Conn_01x15, J3 CONN_02x16_PIN_SMD_Counter_Cl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, J4 Conn_01x03_Male, J5 DX07S016JA1R1500, SW1 SPST_SWITCH_SMD_4P,4.1x5.4mm, U1 TXS0108EPW, U3 TXS0108EPW, U4 TXS0108EPW

Commit message: Autogeneration tools
Connections:
- net labels added: 5VCC
- wire segments 210 -> 214
Changed lines of the file:
@@
 Sheet 1 1
 Title "ESP32 BreakoutBoard 5V"
-Date "2025-09-19"
+Date "2025-10-30"
 Rev "1.2"
 Comp "RetroBit Lab"
@@
 Wire Wire Line
 	9725 5250 9950 5250
-$Comp
-L power:+5V #PWR0127
-U 1 1 68C2BC13
-P 10325 4225
-F 0 "#PWR0127" H 10325 4075 50  0001 C CNN
-F 1 "+5V" H 10340 4398 50  0000 C CNN
-F 2 "" H 10325 4225 50  0001 C CNN
-F 3 "" H 10325 4225 50  0001 C CNN
-	1    10325 4225
-	1    0    0    -1
-$EndComp
 Wire Wire Line
 	9725 4350 10325 4350
@@
 L power:+5V #PWR04
 U 1 1 68959F72
-P 7850 1810
-F 0 "#PWR04" H 7850 1660 50  0001 C CNN
-F 1 "+5V" H 7865 1983 50  0000 C CNN
-F 2 "" H 7850 1810 50  0001 C CNN
-F 3 "" H 7850 1810 50  0001 C CNN
-	1    7850 1810
+P 7640 1745
+F 0 "#PWR04" H 7640 1595 50  0001 C CNN
+F 1 "+5V" H 7640 1885 50  0000 C CNN
+F 2 "" H 7640 1745 50  0001 C CNN
+F 3 "" H 7640 1745 50  0001 C CNN
+	1    7640 1745
 	1    0    0    -1
 $EndComp
@@
 Connection ~ 8035 1850
 Connection ~ 7850 1850
-Wire Wire Line
-	7850 1810 7850 1850
 Wire Wire Line
 	5775 3225 5775 3275
@@
 	-1   0    0    1
 $EndComp
+Wire Wire Line
+	7850 1780 7850 1850
+$Comp
+L power:PWR_FLAG #FLG0103
+U 1 1 69059A03
+P 7490 1795
+F 0 "#FLG0103" H 7490 1870 50  0001 C CNN
+F 1 "PWR_FLAG" H 7490 1968 50  0000 C CNN
+F 2 "" H 7490 1795 50  0001 C CNN
+F 3 "~" H 7490 1795 50  0001 C CNN
+	1    7490 1795
+	-1   0    0    1
+$EndComp
+Wire Wire Line
+	7490 1795 7490 1780
+Wire Wire Line
+	7490 1780 7640 1780
+Wire Wire Line
+	7640 1745 7640 1780
+Connection ~ 7640 1780
+Wire Wire Line
+	7640 1780 7850 1780
+Text Label 7850 1780 0    50   ~ 0
+5VCC
+Text Label 10325 4225 0    50   ~ 0
+5VCC
 $EndSCHEMATC

Commit message: Updated for new pin mappings
Parts:
- removed J3: CONN_02x16_PIN_SMD_Counter_Clockwise, Connector_PinHeader_2.54mm:PinHeader_2x16_P2.54mm_Vertical_SMD, symbol RetroBitLab:CONN_02x16_PIN_SMD_Counter_Clockwise
- added J3: CONN_02x16_PIN_SMD_Counter_Clockwise-RetroBitLab, Connector_PinHeader_2.54mm:PinHeader_2x16_P2.54mm_Vertical_SMD, symbol RetroBitLab:CONN_02x16_PIN_SMD_Counter_Clockwise-RetroBitLab
Changed lines of the file:
@@
 	5745 1400 5875 1400
-$Comp
-L RetroBitLab:CONN_02x16_PIN_SMD_Counter_Clockwise J3
-U 1 1 68D1A2AD
-P 9425 5050
-F 0 "J3" H 9485 5870 50  0000 C CNN
-F 1 "CONN_02x16_PIN_SMD_Counter_Clockwise" H 9485 4130 50  0000 C CNN
-F 2 "Connector_PinHeader_2.54mm:PinHeader_2x16_P2.54mm_Vertical_SMD" H 9425 5050 50  0001 C CNN
-F 3 "https://www.lcsc.com/datasheet/C6332241.pdf" H 9425 5050 50  0001 C CNN
-F 4 "C6332241" H 9425 5050 50  0001 C CNN "LCSC"
-	1    9425 5050
-	1    0    0    -1
-$EndComp
 $Comp
 L CCAP0805:100uF C1
@@
 Text Label 10325 4225 0    50   ~ 0
 5VCC
+$Comp
+L RetroBitLab:CONN_02x16_PIN_SMD_Counter_Clockwise-RetroBitLab J3
+U 1 1 6A276616
+P 9425 5050
+F 0 "J3" H 9470 5885 50  0000 C CNN
+F 1 "CONN_02x16_PIN_SMD_Counter_Clockwise-RetroBitLab" H 9655 4095 50  0000 C CNN
+F 2 "Connector_PinHeader_2.54mm:PinHeader_2x16_P2.54mm_Vertical_SMD" H 9425 5050 50  0001 C CNN
+F 3 "" H 9425 5050 50  0001 C CNN
+F 4 "C6332241" H 9425 5050 50  0001 C CNN "LCSC"
+	1    9425 5050
+	1    0    0    -1
+$EndComp
 $EndSCHEMATC
