File: ESP32-BOBOARD-5V.kicad_pcb (KiCad board)
At the start: 4 copper layers, 100 x 60 mm, 29 parts, among them J1 Conn_01x15, J2 Conn_01x15, J3 CONN_02x16_PIN_SMD_Counter_Cl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, J4 Conn_01x03_Male, J5 DX07S016JA1R1500, SW1 SPST_SWITCH_SMD_4P,4.1x5.4mm, U1 TXS0108EPW, U3 TXS0108EPW, U4 TXS0108EPW

Commit message: Updated for new pin mappings
Parts:
- J3: value CONN_02x16_PIN_SMD_Counter_Clockwise -> CONN_02x16_PIN_SMD_Counter_Clockwise-RetroBitLab
